Commit message: basket now spawning

File: urdf/basket/basket.urdf (robot description, URDF)
Before this commit: robot basket, 1 links, 0 joints
Links:
- removed link basket_link_86
- added link basket_link_368, mass 1; collision mesh filename=package://liquid_pickup/meshes/basket/Basket_V2.stl scale=0.95 0.95 0.95; visual mesh filename=package://liquid_pickup/meshes/basket/Basket_V2.stl scale=0.95 0.95 0.95
