Commit message: also spawning a swab mimicker

File: urdf/swab_container/swab_container.urdf.xacro (robot description, xacro)
@@ -1,8 +1,8 @@
 <?xml version="1.0"?>
-<robot name="basket" xmlns:xacro="http://www.ros.org/wiki/xacro">
+<robot name="swab_container" xmlns:xacro="http://www.ros.org/wiki/xacro">
   <xacro:property name="PI" value="3.1415926535897931"/>
-  <xacro:arg name="basket_link_id" default="basket_link"/>
-  <xacro:macro name="basket" params="prefix parent link_id">
-    <material name="basket_green">
+  <xacro:arg name="swab_container_link_id" default="swab_container_link"/>
+  <xacro:macro name="swab_container" params="prefix parent link_id">
+    <material name="swab_container_green">
       <color rgba="0 1 0 1" />
       <ambient>0 0 0 1</ambient>
@@ -20,5 +20,5 @@
         <origin xyz="0 0 0" rpy="0 0 0" />
         <geometry>
-          <mesh filename="package://liquid_pickup/meshes/basket/Basket_V2.stl" scale="0.95 0.95 0.95" />
+          <mesh filename="package://liquid_pickup/meshes/swab_container/Basket_V2.stl" scale="0.95 0.95 0.95" />
         </geometry>
         <material name="darkgrey">
@@ -29,5 +29,5 @@
         <origin xyz="0 0 0" rpy="0 0 0" />
         <geometry>
-          <mesh filename="package://liquid_pickup/meshes/basket/Basket_V2.stl" scale="0.95 0.95 0.95" />
+          <mesh filename="package://liquid_pickup/meshes/swab_container/Basket_V2.stl" scale="0.95 0.95 0.95" />
         </geometry>
       </collision>
@@ -37,4 +37,4 @@
     </gazebo>
   </xacro:macro>
-  <xacro:basket prefix="summit" parent="base_footprint" link_id="$(arg basket_link_id)" />
+  <xacro:swab_container prefix="summit" parent="base_footprint" link_id="$(arg swab_container_link_id)" />
 </robot>
